File: 996_oil_temp_gauge/version2/version2.kicad_sch (KiCad schematic)
At the start: 15 parts, among them J1 Screw_Terminal_01x01, J2 Screw_Terminal_01x01, J3 Screw_Terminal_01x01, J4 Screw_Terminal_01x01, SW1 SW_SPDT, U1 L7805, U3 MCP6002-xP, U4 ATtiny85-20P

Commit message: Updated schematics
Parts:
- J1: value Screw_Terminal_01x01 -> ECU input
- J2: value Screw_Terminal_01x01 -> Gauge S
- J3: value Screw_Terminal_01x01 -> Gauge V-
- J4: value Screw_Terminal_01x01 -> Gauge V+
Connections:
- net at J1.1 (Pin_1): now also SW1.1 (A); no longer SW1.3 (C)
- net at RV1.2: now also SW1.3 (C); no longer SW1.1 (A)
Other:
- title: (none) -> Porsche 996 VDO Vision Oil Tempearature Gauge Driver
- moved on the sheet: C1, C2, C3, J1, J2, J3, J4, R1, R2, R3, RV1, SW1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
